File: energy_meter/energy_meter.kicad_sch (KiCad schematic)
At the start: 26 parts

Commit message: Added library components for Energy Meter
Parts:
- removed C1, C2, C4: 1nF, symbol The_Parts_Library:C
- removed C3: 22uF, symbol The_Parts_Library:C
- removed D1, D2, D3, D4, D5, D6, D7: D, symbol Device:D
- removed I1: ISIN, symbol Simulation_SPICE:ISIN
- removed R1: 100, symbol Device:R
- removed R12, R4: 6.8k, symbol Device:R
- removed R13: 22, symbol Device:R
- removed R14, R2: 1.1Meg, symbol Device:R
- removed R3: 20k, symbol Device:R
- removed R5: 21.3, symbol Device:R
- removed R6: 12k, symbol Device:R
- removed R7: 62k, symbol Device:R
- removed R9: 3.3k, symbol Device:R
- removed V1: 3, symbol Simulation_SPICE:VDC
- removed V2: 1.8, symbol Simulation_SPICE:VDC
- removed V3: VSIN, symbol Simulation_SPICE:VSIN

Commit message: Board ready to order
Parts:
- added GFX101: ~, The_Parts_Library:Snaily, symbol The_Parts_Library:Gfx_Snaily
- added J101: ~, The_Parts_Library:WAGO_2060-852998-404, symbol The_Parts_Library:J_2060-852/998-404_PWR
Connections:
- new net Power/AC.Line: J101.1, J101.3
- new net Power/AC.Neutral: J101.2, J101.4
Other:
- added sheet HMI (HMI.kicad_sch)
- added sheet Microcontroller (mcu.kicad_sch)
- added sheet Power (power.kicad_sch)
- added sheet Radio (radio.kicad_sch)
- added sheet VSense - ISense (vsense-isense.kicad_sch)
- title: (none) -> Energy Meter
