File: energy_meter/HMI.kicad_sch (KiCad schematic)
At the start: 8 parts

Commit message: Created build outputs for energy-meter rev0
Parts:
- J501: Supplier Part Number 4086 -> 2057-PH1-13-UA-ND
Changed lines of the file:
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@@
 			)
 		)
-		(property "Supplier Part Number" "4086"
+		(property "Supplier Part Number" "2057-PH1-13-UA-ND"
 			(at 157.48 147.32 0)
 			(effects

Commit message: Added The_R0603_Library containing full YAGEO R0603 E96 family.
Parts:
- R501: symbol The_Parts_Library:R0603_100R -> The_R0603_Library:R0603_100R
- R502: symbol The_Parts_Library:R0603_1k -> The_R0603_Library:R0603_1k
- R503: symbol The_Parts_Library:R0603_10k -> The_R0603_Library:R0603_10k
Changed lines of the file:
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@@
 	)
 	(symbol
-		(lib_id "The_Parts_Library:R0603_100R")
+		(lib_id "The_R0603_Library:R0603_100R")
 		(at 90.17 77.47 90)
 		(unit 1)
@@
 	)
 	(symbol
-		(lib_id "The_Parts_Library:R0603_10k")
+		(lib_id "The_R0603_Library:R0603_10k")
 		(at 165.1 68.58 0)
 		(unit 1)
@@
 	)
 	(symbol
-		(lib_id "The_Parts_Library:R0603_1k")
+		(lib_id "The_R0603_Library:R0603_1k")
 		(at 100.33 72.39 0)
 		(unit 1)

Commit message: Added The_C0603_Library with Murata GCM188 family of capacitors
Parts:
- C501: symbol The_Parts_Library:C0603_100nF_100V_X7R -> The_C0603_Library:C0603_100nF_100V_X7R
Changed lines of the file:
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@@
 	)
 	(symbol
-		(lib_id "The_Parts_Library:C0603_100nF_100V_X7R")
+		(lib_id "The_C0603_Library:C0603_100nF_100V_X7R")
 		(at 165.1 78.74 0)
 		(unit 1)
