File: energy_meter/mcu.kicad_sch (KiCad schematic)
At the start: 16 parts, among them X401 38.4MHz, X402 32.768kHz

Commit message: Added The_C0603_Library with Murata GCM188 family of capacitors
Parts:
- C402, C403, C407: symbol The_Parts_Library:C0603_1uF_25V_X7R -> The_C0603_Library:C0603_1uF_25V_X7R
- C404, C405, C406, C408, C409, C411: symbol The_Parts_Library:C0603_100nF_100V_X7R -> The_C0603_Library:C0603_100nF_100V_X7R
Changed lines of the file:
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@@
 	)
 	(symbol
-		(lib_id "The_Parts_Library:C0603_100nF_100V_X7R")
+		(lib_id "The_C0603_Library:C0603_100nF_100V_X7R")
 		(at 163.83 71.12 0)
 		(unit 1)
@@
 	)
 	(symbol
-		(lib_id "The_Parts_Library:C0603_100nF_100V_X7R")
+		(lib_id "The_C0603_Library:C0603_100nF_100V_X7R")
 		(at 175.26 71.12 0)
 		(unit 1)
@@
 	)
 	(symbol
-		(lib_id "The_Parts_Library:C0603_100nF_100V_X7R")
+		(lib_id "The_C0603_Library:C0603_100nF_100V_X7R")
 		(at 96.52 74.93 0)
 		(unit 1)
@@
 	)
 	(symbol
-		(lib_id "The_Parts_Library:C0603_100nF_100V_X7R")
+		(lib_id "The_C0603_Library:C0603_100nF_100V_X7R")
 		(at 96.52 63.5 0)
 		(unit 1)
@@
 	)
 	(symbol
-		(lib_id "The_Parts_Library:C0603_100nF_100V_X7R")
+		(lib_id "The_C0603_Library:C0603_100nF_100V_X7R")
 		(at 186.69 71.12 0)
 		(unit 1)
@@
 	)
 	(symbol
-		(lib_id "The_Parts_Library:C0603_100nF_100V_X7R")
+		(lib_id "The_C0603_Library:C0603_100nF_100V_X7R")
 		(at 96.52 87.63 0)
 		(unit 1)
@@
 	)
 	(symbol
-		(lib_id "The_Parts_Library:C0603_1uF_25V_X7R")
+		(lib_id "The_C0603_Library:C0603_1uF_25V_X7R")
 		(at 82.55 87.63 0)
 		(unit 1)
@@
 	)
 	(symbol
-		(lib_id "The_Parts_Library:C0603_1uF_25V_X7R")
+		(lib_id "The_C0603_Library:C0603_1uF_25V_X7R")
 		(at 82.55 74.93 0)
 		(unit 1)
@@
 	)
 	(symbol
-		(lib_id "The_Parts_Library:C0603_1uF_25V_X7R")
+		(lib_id "The_C0603_Library:C0603_1uF_25V_X7R")
 		(at 158.75 92.71 90)
 		(unit 1)
