File: energy_meter/power.kicad_sch (KiCad schematic)
At the start: 27 parts

Commit message: Added The_R0603_Library containing full YAGEO R0603 E96 family.
Parts:
- R203: symbol The_Parts_Library:R0603_100k -> The_R0603_Library:R0603_100k
- R205: symbol The_Parts_Library:R0603_10R -> The_R0603_Library:R0603_10R
- R206: symbol The_Parts_Library:R0603_82k -> The_R0603_Library:R0603_82k
- R207: symbol The_Parts_Library:R0603_10k -> The_R0603_Library:R0603_10k
- R208: symbol The_Parts_Library:R0603_40.2k -> The_R0603_Library:R0603_40.2k
Changed lines of the file:
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@@
 	)
 	(symbol
-		(lib_id "The_Parts_Library:R0603_10R")
+		(lib_id "The_R0603_Library:R0603_10R")
 		(at 133.35 138.43 90)
 		(unit 1)
@@
 	)
 	(symbol
-		(lib_id "The_Parts_Library:R0603_10k")
+		(lib_id "The_R0603_Library:R0603_10k")
 		(at 140.97 170.18 0)
 		(unit 1)
@@
 	)
 	(symbol
-		(lib_id "The_Parts_Library:R0603_82k")
+		(lib_id "The_R0603_Library:R0603_82k")
 		(at 134.62 163.83 90)
 		(unit 1)
@@
 	)
 	(symbol
-		(lib_id "The_Parts_Library:R0603_40.2k")
+		(lib_id "The_R0603_Library:R0603_40.2k")
 		(at 147.32 163.83 90)
 		(unit 1)
@@
 	)
 	(symbol
-		(lib_id "The_Parts_Library:R0603_100k")
+		(lib_id "The_R0603_Library:R0603_100k")
 		(at 104.14 142.24 0)
 		(unit 1)

Commit message: Added The_C0603_Library with Murata GCM188 family of capacitors
Parts:
- C202: symbol The_Parts_Library:C0603_100nF_100V_X7R -> The_C0603_Library:C0603_100nF_100V_X7R
- C204: symbol The_Parts_Library:C0603_1uF_25V_X7R -> The_C0603_Library:C0603_1uF_25V_X7R
- C205: symbol The_Parts_Library:C0603_15pF_100V_C0G -> The_C0603_Library:C0603_15pF_100V_C0G
Changed lines of the file:
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@@
 	)
 	(symbol
-		(lib_id "The_Parts_Library:C0603_1uF_25V_X7R")
+		(lib_id "The_C0603_Library:C0603_1uF_25V_X7R")
 		(at 140.97 138.43 90)
 		(unit 1)
@@
 	)
 	(symbol
-		(lib_id "The_Parts_Library:C0603_15pF_100V_C0G")
+		(lib_id "The_C0603_Library:C0603_15pF_100V_C0G")
 		(at 147.32 154.94 90)
 		(unit 1)
@@
 	)
 	(symbol
-		(lib_id "The_Parts_Library:C0603_100nF_100V_X7R")
+		(lib_id "The_C0603_Library:C0603_100nF_100V_X7R")
 		(at 92.71 142.24 0)
 		(unit 1)
