File: energy_meter/radio.kicad_sch (KiCad schematic)
At the start: 28 parts, among them X601 27MHz

Commit message: Added The_R0603_Library containing full YAGEO R0603 E96 family.
Parts:
- R601: symbol The_Parts_Library:R0603_56k -> The_R0603_Library:R0603_56k
Changed lines of the file:
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@@
 	)
 	(symbol
-		(lib_id "The_Parts_Library:R0603_56k")
+		(lib_id "The_R0603_Library:R0603_56k")
 		(at 114.3 116.84 0)
 		(unit 1)

Commit message: Added The_C0603_Library with Murata GCM188 family of capacitors
Parts:
- C601, C602, C603, C604, C605, C606, C607: symbol The_Parts_Library:C0603_100nF_100V_X7R -> The_C0603_Library:C0603_100nF_100V_X7R
- C608, C609: symbol The_Parts_Library:C0603_15pF_100V_C0G -> The_C0603_Library:C0603_15pF_100V_C0G
- C610, C616, C617: symbol The_Parts_Library:C0603_1pF_100V_C0G -> The_C0603_Library:C0603_1pF_100V_C0G
- C611, C613: symbol The_Parts_Library:C0603_1.5pF_100V_C0G -> The_C0603_Library:C0603_1.5pF_100V_C0G
- C612, C615: symbol The_Parts_Library:C0603_100pF_100V_C0G -> The_C0603_Library:C0603_100pF_100V_C0G
- C614: symbol The_Parts_Library:C0603_3.3pF_100V_C0G -> The_C0603_Library:C0603_3.3pF_100V_C0G
Changed lines of the file:
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@@
 	)
 	(symbol
-		(lib_id "The_Parts_Library:C0603_100nF_100V_X7R")
+		(lib_id "The_C0603_Library:C0603_100nF_100V_X7R")
 		(at 86.36 82.55 0)
 		(unit 1)
@@
 	)
 	(symbol
-		(lib_id "The_Parts_Library:C0603_100nF_100V_X7R")
+		(lib_id "The_C0603_Library:C0603_100nF_100V_X7R")
 		(at 35.56 69.85 0)
 		(unit 1)
@@
 	)
 	(symbol
-		(lib_id "The_Parts_Library:C0603_1.5pF_100V_C0G")
+		(lib_id "The_C0603_Library:C0603_1.5pF_100V_C0G")
 		(at 203.2 72.39 90)
 		(unit 1)
@@
 	)
 	(symbol
-		(lib_id "The_Parts_Library:C0603_100pF_100V_C0G")
+		(lib_id "The_C0603_Library:C0603_100pF_100V_C0G")
 		(at 242.57 77.47 90)
 		(unit 1)
@@
 	)
 	(symbol
-		(lib_id "The_Parts_Library:C0603_100nF_100V_X7R")
+		(lib_id "The_C0603_Library:C0603_100nF_100V_X7R")
 		(at 66.04 77.47 0)
 		(unit 1)
@@
 	)
 	(symbol
-		(lib_id "The_Parts_Library:C0603_100nF_100V_X7R")
+		(lib_id "The_C0603_Library:C0603_100nF_100V_X7R")
 		(at 45.72 72.39 0)
 		(unit 1)
@@
 	)
 	(symbol
-		(lib_id "The_Parts_Library:C0603_1pF_100V_C0G")
+		(lib_id "The_C0603_Library:C0603_1pF_100V_C0G")
 		(at 180.34 77.47 0)
 		(unit 1)
@@
 	)
 	(symbol
-		(lib_id "The_Parts_Library:C0603_100nF_100V_X7R")
+		(lib_id "The_C0603_Library:C0603_100nF_100V_X7R")
 		(at 76.2 80.01 0)
 		(unit 1)
@@
 	)
 	(symbol
-		(lib_id "The_Parts_Library:C0603_100nF_100V_X7R")
+		(lib_id "The_C0603_Library:C0603_100nF_100V_X7R")
 		(at 96.52 85.09 0)
 		(unit 1)
@@
 	)
 	(symbol
-		(lib_id "The_Parts_Library:C0603_1pF_100V_C0G")
+		(lib_id "The_C0603_Library:C0603_1pF_100V_C0G")
 		(at 256.54 77.47 90)
 		(unit 1)
@@
 	)
 	(symbol
-		(lib_id "The_Parts_Library:C0603_100nF_100V_X7R")
+		(lib_id "The_C0603_Library:C0603_100nF_100V_X7R")
 		(at 55.88 74.93 0)
 		(unit 1)
@@
 	)
 	(symbol
-		(lib_id "The_Parts_Library:C0603_15pF_100V_C0G")
+		(lib_id "The_C0603_Library:C0603_15pF_100V_C0G")
 		(at 165.1 97.79 90)
 		(unit 1)
@@
 	)
 	(symbol
-		(lib_id "The_Parts_Library:C0603_1pF_100V_C0G")
+		(lib_id "The_C0603_Library:C0603_1pF_100V_C0G")
 		(at 248.92 83.82 0)
 		(unit 1)
@@
 	)
 	(symbol
-		(lib_id "The_Parts_Library:C0603_15pF_100V_C0G")
+		(lib_id "The_C0603_Library:C0603_15pF_100V_C0G")
 		(at 165.1 87.63 90)
 		(unit 1)
@@
 	)
 	(symbol
-		(lib_id "The_Parts_Library:C0603_1.5pF_100V_C0G")
+		(lib_id "The_C0603_Library:C0603_1.5pF_100V_C0G")
 		(at 184.15 87.63 180)
 		(unit 1)
@@
 	)
 	(symbol
-		(lib_id "The_Parts_Library:C0603_100pF_100V_C0G")
+		(lib_id "The_C0603_Library:C0603_100pF_100V_C0G")
 		(at 194.31 99.06 0)
 		(unit 1)
@@
 	)
 	(symbol
-		(lib_id "The_Parts_Library:C0603_3.3pF_100V_C0G")
+		(lib_id "The_C0603_Library:C0603_3.3pF_100V_C0G")
 		(at 226.06 83.82 0)
 		(unit 1)
