File: energy_meter/vsense-isense.kicad_sch (KiCad schematic)
At the start: 16 parts

Commit message: Added The_R0603_Library containing full YAGEO R0603 E96 family.
Parts:
- R301: symbol The_Parts_Library:R0603_12k -> The_R0603_Library:R0603_12k
- R303: symbol The_Parts_Library:R0603_62k -> The_R0603_Library:R0603_62k
- R304: symbol The_Parts_Library:R0603_3.3k -> The_R0603_Library:R0603_3.3k
- R307: symbol The_Parts_Library:R0603_20k -> The_R0603_Library:R0603_20k
- R308, R309: symbol The_Parts_Library:R0603_6.8k -> The_R0603_Library:R0603_6.8k
Changed lines of the file:
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@@
 	)
 	(symbol
-		(lib_id "The_Parts_Library:R0603_3.3k")
+		(lib_id "The_R0603_Library:R0603_3.3k")
 		(at 115.57 62.23 90)
 		(unit 1)
@@
 	)
 	(symbol
-		(lib_id "The_Parts_Library:R0603_6.8k")
+		(lib_id "The_R0603_Library:R0603_6.8k")
 		(at 129.54 111.76 0)
 		(unit 1)
@@
 	)
 	(symbol
-		(lib_id "The_Parts_Library:R0603_62k")
+		(lib_id "The_R0603_Library:R0603_62k")
 		(at 104.14 80.01 0)
 		(unit 1)
@@
 	)
 	(symbol
-		(lib_id "The_Parts_Library:R0603_12k")
+		(lib_id "The_R0603_Library:R0603_12k")
 		(at 104.14 53.34 0)
 		(unit 1)
@@
 	)
 	(symbol
-		(lib_id "The_Parts_Library:R0603_20k")
+		(lib_id "The_R0603_Library:R0603_20k")
 		(at 125.73 68.58 0)
 		(unit 1)
@@
 	)
 	(symbol
-		(lib_id "The_Parts_Library:R0603_6.8k")
+		(lib_id "The_R0603_Library:R0603_6.8k")
 		(at 130.81 149.86 0)
 		(unit 1)

Commit message: Added The_C0603_Library with Murata GCM188 family of capacitors
Parts:
- C301, C302, C303: symbol The_Parts_Library:C0603_1nF_50V_C0G -> The_C0603_Library:C0603_1nF_50V_C0G
Changed lines of the file:
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@@
 	)
 	(symbol
-		(lib_id "The_Parts_Library:C0603_1nF_50V_C0G")
+		(lib_id "The_C0603_Library:C0603_1nF_50V_C0G")
 		(at 139.7 68.58 0)
 		(unit 1)
@@
 	)
 	(symbol
-		(lib_id "The_Parts_Library:C0603_1nF_50V_C0G")
+		(lib_id "The_C0603_Library:C0603_1nF_50V_C0G")
 		(at 140.97 149.86 0)
 		(unit 1)
@@
 	)
 	(symbol
-		(lib_id "The_Parts_Library:C0603_1nF_50V_C0G")
+		(lib_id "The_C0603_Library:C0603_1nF_50V_C0G")
 		(at 140.97 111.76 0)
 		(unit 1)
