File: Syncd_EFM32s/Syncd_EFM32s.kicad_sch (KiCad schematic)
At the start: 37 parts, among them X101 38.4MHz, X102 32.768kHz

Commit message: Added The_R0603_Library containing full YAGEO R0603 E96 family.
Parts:
- R101, R102: symbol The_Parts_Library:R0603_1k -> The_R0603_Library:R0603_1k
Changed lines of the file:
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@@
 	)
 	(symbol
-		(lib_id "The_Parts_Library:R0603_1k")
+		(lib_id "The_R0603_Library:R0603_1k")
 		(at 33.02 166.37 0)
 		(unit 1)
@@
 	)
 	(symbol
-		(lib_id "The_Parts_Library:R0603_1k")
+		(lib_id "The_R0603_Library:R0603_1k")
 		(at 123.19 161.29 0)
 		(unit 1)

Commit message: Added The_C0603_Library with Murata GCM188 family of capacitors
Parts:
- C104, C105, C106, C107, C108, C118: symbol The_Parts_Library:C0603_1uF_25V_X7R -> The_C0603_Library:C0603_1uF_25V_X7R
- C109, C110, C111, C112, C113, C114, C115, C116, C117, C119, C120, C121: symbol The_Parts_Library:C0603_100nF_100V_X7R -> The_C0603_Library:C0603_100nF_100V_X7R
Changed lines of the file:
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@@
 	)
 	(symbol
-		(lib_id "The_Parts_Library:C0603_100nF_100V_X7R")
+		(lib_id "The_C0603_Library:C0603_100nF_100V_X7R")
 		(at 102.87 26.67 0)
 		(mirror y)
@@
 	)
 	(symbol
-		(lib_id "The_Parts_Library:C0603_1uF_25V_X7R")
+		(lib_id "The_C0603_Library:C0603_1uF_25V_X7R")
 		(at 151.13 45.72 0)
 		(unit 1)
@@
 	)
 	(symbol
-		(lib_id "The_Parts_Library:C0603_1uF_25V_X7R")
+		(lib_id "The_C0603_Library:C0603_1uF_25V_X7R")
 		(at 93.98 63.5 90)
 		(unit 1)
@@
 	)
 	(symbol
-		(lib_id "The_Parts_Library:C0603_100nF_100V_X7R")
+		(lib_id "The_C0603_Library:C0603_100nF_100V_X7R")
 		(at 232.41 25.4 0)
 		(mirror y)
@@
 	)
 	(symbol
-		(lib_id "The_Parts_Library:C0603_100nF_100V_X7R")
+		(lib_id "The_C0603_Library:C0603_100nF_100V_X7R")
 		(at 163.83 35.56 0)
 		(unit 1)
@@
 	)
 	(symbol
-		(lib_id "The_Parts_Library:C0603_1uF_25V_X7R")
+		(lib_id "The_C0603_Library:C0603_1uF_25V_X7R")
 		(at 223.52 62.23 90)
 		(unit 1)
@@
 	)
 	(symbol
-		(lib_id "The_Parts_Library:C0603_100nF_100V_X7R")
+		(lib_id "The_C0603_Library:C0603_100nF_100V_X7R")
 		(at 232.41 35.56 0)
 		(mirror y)
@@
 	)
 	(symbol
-		(lib_id "The_Parts_Library:C0603_1uF_25V_X7R")
+		(lib_id "The_C0603_Library:C0603_1uF_25V_X7R")
 		(at 151.13 57.15 0)
 		(unit 1)
@@
 	)
 	(symbol
-		(lib_id "The_Parts_Library:C0603_100nF_100V_X7R")
+		(lib_id "The_C0603_Library:C0603_100nF_100V_X7R")
 		(at 30.48 46.99 0)
 		(unit 1)
@@
 	)
 	(symbol
-		(lib_id "The_Parts_Library:C0603_100nF_100V_X7R")
+		(lib_id "The_C0603_Library:C0603_100nF_100V_X7R")
 		(at 163.83 57.15 0)
 		(unit 1)
@@
 	)
 	(symbol
-		(lib_id "The_Parts_Library:C0603_1uF_25V_X7R")
+		(lib_id "The_C0603_Library:C0603_1uF_25V_X7R")
 		(at 17.78 58.42 0)
 		(unit 1)
@@
 	)
 	(symbol
-		(lib_id "The_Parts_Library:C0603_100nF_100V_X7R")
+		(lib_id "The_C0603_Library:C0603_100nF_100V_X7R")
 		(at 232.41 45.72 0)
 		(mirror y)
@@
 	)
 	(symbol
-		(lib_id "The_Parts_Library:C0603_100nF_100V_X7R")
+		(lib_id "The_C0603_Library:C0603_100nF_100V_X7R")
 		(at 163.83 45.72 0)
 		(unit 1)
@@
 	)
 	(symbol
-		(lib_id "The_Parts_Library:C0603_100nF_100V_X7R")
+		(lib_id "The_C0603_Library:C0603_100nF_100V_X7R")
 		(at 102.87 36.83 0)
 		(mirror y)
@@
 	)
 	(symbol
-		(lib_id "The_Parts_Library:C0603_100nF_100V_X7R")
+		(lib_id "The_C0603_Library:C0603_100nF_100V_X7R")
 		(at 30.48 36.83 0)
 		(unit 1)
@@
 	)
 	(symbol
-		(lib_id "The_Parts_Library:C0603_1uF_25V_X7R")
+		(lib_id "The_C0603_Library:C0603_1uF_25V_X7R")
 		(at 17.78 46.99 0)
 		(unit 1)
@@
 	)
 	(symbol
-		(lib_id "The_Parts_Library:C0603_100nF_100V_X7R")
+		(lib_id "The_C0603_Library:C0603_100nF_100V_X7R")
 		(at 30.48 58.42 0)
 		(unit 1)
@@
 	)
 	(symbol
-		(lib_id "The_Parts_Library:C0603_100nF_100V_X7R")
+		(lib_id "The_C0603_Library:C0603_100nF_100V_X7R")
 		(at 102.87 46.99 0)
 		(mirror y)
